File: design/KicadDesign/KicadDesign.kicad_pcb (KiCad board)
At the start: 2 copper layers, 39.3 x 11.8 mm, 8 parts, among them J1 Servo0, J2 Servo1, J3 Servo2, J4 Servo3, J5 ORANGE, J6 Source

Commit message: feat: add ground plane
Routing:
- added copper zone on B.Cu, net GND
Changed lines of the file:
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@@
 		(net "/PWM3")
+	)
+	(zone
+		(net "GND")
+		(layer "B.Cu")
+		(hatch edge 0.5)
+		(connect_pads
+			(clearance 0.5)
+		)
+		(min_thickness 0.25)
+		(fill yes
+			(thermal_gap 0.5)
+			(thermal_bridge_width 0.5)
+			(island_removal_mode 0)
+		)
+		(polygon
+			(pts
+				(xy 103.124 69.3928) (xy 103.124 68.9864) (xy 103.7336 68.9864) (xy 103.7336 81.3816) (xy 63.5508 81.3816)
+				(xy 63.5508 69.3928)
+			)
+		)
 	)
 	(embedded_fonts no)
